File: SPH0641LU.sch (KiCad schematic (older format))
At the start: 5 parts, among them P1 CONN_01X05, U1 SPH0641LU4H

Commit message: copied 16 microphones
Parts:
- removed R1, R2: R, generic:generic-SMD1608, symbol R
- added C10, C11, C12, C13, C14, C15, C16, C2, C3, C4, C5, C6, C7, C8, C9: 100nF, generic:generic-SMD1608, symbol Device:C
- added U10, U11, U12, U13, U14, U15, U16, U2, U3, U4, U5, U6, U7, U8, U9: SPH0641LU4H, SPH0641LU4H:SPH0641LU4H, symbol SPH0641LU-rescue:SPH0641LU4H
- C1: value C -> 100nF; symbol C -> Device:C
- P1: footprint pin-head:pinhead-1X05 -> SIL-6; symbol CONN_01X05 -> SPH0641LU-rescue:CONN_01X05
- U1: symbol SPH0641LU4H -> SPH0641LU-rescue:SPH0641LU4H
Connections:
- net CLK: now also U10.4 (CLOCK), U11.4 (CLOCK), U12.4 (CLOCK), U13.4 (CLOCK), U14.4 (CLOCK), U15.4 (CLOCK), U16.4 (CLOCK), U2.4 (CLOCK), U3.4 (CLOCK), U4.4 (CLOCK), U5.4 (CLOCK), U6.4 (CLOCK), U7.4 (CLOCK), U8.4 (CLOCK), U9.4 (CLOCK)
- net DATA: no longer U1.1 (DATA)
- net GND: now also C10.2, C11.2, C12.2, C13.2, C14.2, C15.2, C16.2, C2.2, C3.2, C4.2, C5.2, C6.2, C7.2, C8.2, C9.2, U10.3 (GROUND), U11.3 (GROUND), U12.3 (GROUND), U13.3 (GROUND), U14.3 (GROUND), U15.3 (GROUND), U16.3 (GROUND), U2.3 (GROUND), U3.3 (GROUND), U4.3 (GROUND), U5.3 (GROUND), U6.3 (GROUND), U7.3 (GROUND), U8.3 (GROUND), U9.3 (GROUND)
- net LRSEL: no longer U1.2 (SELECT)
- net VDD renamed +3V3
- net +3V3: now also C10.1, C11.1, C12.1, C13.1, C14.1, C15.1, C16.1, C2.1, C3.1, C4.1, C5.1, C6.1, C7.1, C8.1, C9.1, U10.5 (VDD), U11.5 (VDD), U12.5 (VDD), U13.5 (VDD), U14.5 (VDD), U15.5 (VDD), U16.5 (VDD), U2.5 (VDD), U3.5 (VDD), U4.5 (VDD), U5.5 (VDD), U6.5 (VDD), U7.5 (VDD), U8.5 (VDD), U9.5 (VDD)
- new net DATA[0]: U1.1 (DATA), U11.1 (DATA), U13.1 (DATA), U15.1 (DATA), U3.1 (DATA), U5.1 (DATA), U7.1 (DATA), U9.1 (DATA)
- new net DATA[1]: U10.1 (DATA), U12.1 (DATA), U14.1 (DATA), U16.1 (DATA), U2.1 (DATA), U4.1 (DATA), U6.1 (DATA), U8.1 (DATA)
- new net LRSEL_L: U10.2 (SELECT), U12.2 (SELECT), U14.2 (SELECT), U16.2 (SELECT), U2.2 (SELECT), U4.2 (SELECT), U6.2 (SELECT), U8.2 (SELECT)
- new net SEL_RISE: U1.2 (SELECT), U11.2 (SELECT), U13.2 (SELECT), U15.2 (SELECT), U3.2 (SELECT), U5.2 (SELECT), U7.2 (SELECT), U9.2 (SELECT)
Other:
- moved on the sheet: C1, P1, U1

Commit message: moved changes from rescue library to default libraries
Parts:
- P1: symbol SPH0641LU-rescue:CONN_01X05 -> Connector_Generic:Conn_01x05
- U1, U10, U11, U12, U13, U14, U15, U16, U2, U3, U4, U5, U6, U7, U8, U9: symbol SPH0641LU-rescue:SPH0641LU4H -> sph0641lu4h:SPH0641LU4H
Changed lines of the file:
@@
 $EndDescr
 $Comp
-L SPH0641LU-rescue:CONN_01X05 P1
+L Connector_Generic:Conn_01x05 P1
 U 1 1 58F35D98
 P 8550 4800
@@
 F 1 "CONN_01X05" V 8650 4800 50  0000 C CNN
 F 2 "SIL-6" H 8550 4800 50  0001 C CNN
-F 3 "" H 8550 4800 50  0000 C CNN
+F 3 "~" H 8550 4800 50  0000 C CNN
 	1    8550 4800
 	-1   0    0    -1
@@
 F 1 "100nF" H 1325 1550 50  0000 L CNN
 F 2 "generic:generic-SMD1608" H 1338 1500 50  0001 C CNN
-F 3 "" H 1300 1650 50  0000 C CNN
+F 3 "~" H 1300 1650 50  0000 C CNN
 	1    1300 1650
 	1    0    0    -1
@@
 	1300 1800 1300 1850
 $Comp
-L SPH0641LU-rescue:SPH0641LU4H U1
+L sph0641lu4h:SPH0641LU4H U1
 U 1 1 58F360D1
 P 2050 1350
@@
 F 1 "100nF" H 2975 1550 50  0000 L CNN
 F 2 "generic:generic-SMD1608" H 2988 1500 50  0001 C CNN
-F 3 "" H 2950 1650 50  0000 C CNN
+F 3 "~" H 2950 1650 50  0000 C CNN
 	1    2950 1650
 	1    0    0    -1
@@
 	2950 1800 2950 1850
 $Comp
-L SPH0641LU-rescue:SPH0641LU4H U2
+L sph0641lu4h:SPH0641LU4H U2
 U 1 1 5D1AB540
 P 3700 1350
@@
 F 1 "100nF" H 4675 1550 50  0000 L CNN
 F 2 "generic:generic-SMD1608" H 4688 1500 50  0001 C CNN
-F 3 "" H 4650 1650 50  0000 C CNN
+F 3 "~" H 4650 1650 50  0000 C CNN
 	1    4650 1650
 	1    0    0    -1
@@
 	4650 1800 4650 1850
 $Comp
-L SPH0641LU-rescue:SPH0641LU4H U3
+L sph0641lu4h:SPH0641LU4H U3
 U 1 1 5D1BA6CB
 P 5400 1350
@@
 F 1 "100nF" H 6325 1550 50  0000 L CNN
 F 2 "generic:generic-SMD1608" H 6338 1500 50  0001 C CNN
-F 3 "" H 6300 1650 50  0000 C CNN
+F 3 "~" H 6300 1650 50  0000 C CNN
 	1    6300 1650
 	1    0    0    -1
@@
 	6300 1800 6300 1850
 $Comp
-L SPH0641LU-rescue:SPH0641LU4H U4
+L sph0641lu4h:SPH0641LU4H U4
 U 1 1 5D1BA6F5
 P 7050 1350
@@
 F 1 "100nF" H 1325 3100 50  0000 L CNN
 F 2 "generic:generic-SMD1608" H 1338 3050 50  0001 C CNN
-F 3 "" H 1300 3200 50  0000 C CNN
+F 3 "~" H 1300 3200 50  0000 C CNN
 	1    1300 3200
 	1    0    0    -1
@@
 	1300 3350 1300 3400
 $Comp
-L SPH0641LU-rescue:SPH0641LU4H U5
+L sph0641lu4h:SPH0641LU4H U5
 U 1 1 5D1CFD0F
 P 2050 2900
@@
 F 1 "100nF" H 2975 3100 50  0000 L CNN
 F 2 "generic:generic-SMD1608" H 2988 3050 50  0001 C CNN
-F 3 "" H 2950 3200 50  0000 C CNN
+F 3 "~" H 2950 3200 50  0000 C CNN
 	1    2950 3200
 	1    0    0    -1
@@
 	2950 3350 2950 3400
 $Comp
-L SPH0641LU-rescue:SPH0641LU4H U6
+L sph0641lu4h:SPH0641LU4H U6
 U 1 1 5D1CFD39
 P 3700 2900
@@
 F 1 "100nF" H 4675 3100 50  0000 L CNN
 F 2 "generic:generic-SMD1608" H 4688 3050 50  0001 C CNN
-F 3 "" H 4650 3200 50  0000 C CNN
+F 3 "~" H 4650 3200 50  0000 C CNN
 	1    4650 3200
 	1    0    0    -1
@@
 	4650 3350 4650 3400
 $Comp
-L SPH0641LU-rescue:SPH0641LU4H U7
+L sph0641lu4h:SPH0641LU4H U7
 U 1 1 5D1CFD63
 P 5400 2900
@@
 F 1 "100nF" H 6325 3100 50  0000 L CNN
 F 2 "generic:generic-SMD1608" H 6338 3050 50  0001 C CNN
-F 3 "" H 6300 3200 50  0000 C CNN
+F 3 "~" H 6300 3200 50  0000 C CNN
 	1    6300 3200
 	1    0    0    -1
@@
 	6300 3350 6300 3400
 $Comp
-L SPH0641LU-rescue:SPH0641LU4H U8
+L sph0641lu4h:SPH0641LU4H U8
 U 1 1 5D1CFD8D
 P 7050 2900
@@
 F 1 "100nF" H 1325 4650 50  0000 L CNN
 F 2 "generic:generic-SMD1608" H 1338 4600 50  0001 C CNN
-F 3 "" H 1300 4750 50  0000 C CNN
+F 3 "~" H 1300 4750 50  0000 C CNN
 	1    1300 4750
 	1    0    0    -1
@@
 	1300 4900 1300 4950
 $Comp
-L SPH0641LU-rescue:SPH0641LU4H U9
+L sph0641lu4h:SPH0641LU4H U9
 U 1 1 5D2131E2
 P 2050 4450
@@
 F 1 "100nF" H 2975 4650 50  0000 L CNN
 F 2 "generic:generic-SMD1608" H 2988 4600 50  0001 C CNN
-F 3 "" H 2950 4750 50  0000 C CNN
+F 3 "~" H 2950 4750 50  0000 C CNN
 	1    2950 4750
 	1    0    0    -1
@@
 	2950 4900 2950 4950
 $Comp
-L SPH0641LU-rescue:SPH0641LU4H U10
+L sph0641lu4h:SPH0641LU4H U10
 U 1 1 5D21320C
 P 3700 4450
@@
 F 1 "100nF" H 4675 4650 50  0000 L CNN
 F 2 "generic:generic-SMD1608" H 4688 4600 50  0001 C CNN
-F 3 "" H 4650 4750 50  0000 C CNN
+F 3 "~" H 4650 4750 50  0000 C CNN
 	1    4650 4750
 	1    0    0    -1
@@
 	4650 4900 4650 4950
 $Comp
-L SPH0641LU-rescue:SPH0641LU4H U11
+L sph0641lu4h:SPH0641LU4H U11
 U 1 1 5D213236
 P 5400 4450
@@
 F 1 "100nF" H 6325 4650 50  0000 L CNN
 F 2 "generic:generic-SMD1608" H 6338 4600 50  0001 C CNN
-F 3 "" H 6300 4750 50  0000 C CNN
+F 3 "~" H 6300 4750 50  0000 C CNN
 	1    6300 4750
 	1    0    0    -1
@@
 	6300 4900 6300 4950
 $Comp
-L SPH0641LU-rescue:SPH0641LU4H U12
+L sph0641lu4h:SPH0641LU4H U12
 U 1 1 5D213260
 P 7050 4450
@@
 F 1 "100nF" H 1325 6200 50  0000 L CNN
 F 2 "generic:generic-SMD1608" H 1338 6150 50  0001 C CNN
-F 3 "" H 1300 6300 50  0000 C CNN
+F 3 "~" H 1300 6300 50  0000 C CNN
 	1    1300 6300
 	1    0    0    -1
@@
 	1300 6450 1300 6500
 $Comp
-L SPH0641LU-rescue:SPH0641LU4H U13
+L sph0641lu4h:SPH0641LU4H U13
 U 1 1 5D21328A
 P 2050 6000
@@
 F 1 "100nF" H 2975 6200 50  0000 L CNN
 F 2 "generic:generic-SMD1608" H 2988 6150 50  0001 C CNN
-F 3 "" H 2950 6300 50  0000 C CNN
+F 3 "~" H 2950 6300 50  0000 C CNN
 	1    2950 6300
 	1    0    0    -1
@@
 	2950 6450 2950 6500
 $Comp
-L SPH0641LU-rescue:SPH0641LU4H U14
+L sph0641lu4h:SPH0641LU4H U14
 U 1 1 5D2132B4
 P 3700 6000
@@
 F 1 "100nF" H 4675 6200 50  0000 L CNN
 F 2 "generic:generic-SMD1608" H 4688 6150 50  0001 C CNN
-F 3 "" H 4650 6300 50  0000 C CNN
+F 3 "~" H 4650 6300 50  0000 C CNN
 	1    4650 6300
 	1    0    0    -1
@@
 	4650 6450 4650 6500
 $Comp
-L SPH0641LU-rescue:SPH0641LU4H U15
+L sph0641lu4h:SPH0641LU4H U15
 U 1 1 5D2132DE
 P 5400 6000
@@
 F 1 "100nF" H 6325 6200 50  0000 L CNN
 F 2 "generic:generic-SMD1608" H 6338 6150 50  0001 C CNN
-F 3 "" H 6300 6300 50  0000 C CNN
+F 3 "~" H 6300 6300 50  0000 C CNN
 	1    6300 6300
 	1    0    0    -1
@@
 	6300 6450 6300 6500
 $Comp
-L SPH0641LU-rescue:SPH0641LU4H U16
+L sph0641lu4h:SPH0641LU4H U16
 U 1 1 5D213308
 P 7050 6000
